File: design_board/controller_wifi/controller.sch (EAGLE design)
At the start: 67 parts, among them IC1 L293D, IC2 7805DT, IC4 7805TV

Commit message: Изменены платы controller.brd и relay.brd - скорректированы зазоры между платами, оp_amp.brd - добавлено отверстие для прокладки проводки между уровнями. Изменена схема сontroller.sch - добавлены номиналы резисторов обвязки оптопар.
Parts:
- R1, R2, R3, R4, R5: value (none) -> 4,7 kOm
- R10, R6, R7, R8, R9: value (none) -> 1 kOm
Changed lines of the file:
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@@
 <part name="+3V5" library="supply1" deviceset="+3V3" device=""/>
 <part name="+3V6" library="supply1" deviceset="+3V3" device=""/>
-<part name="R1" library="resistor" deviceset="R-EU_" device="0204/5"/>
-<part name="R2" library="resistor" deviceset="R-EU_" device="0204/5"/>
-<part name="R3" library="resistor" deviceset="R-EU_" device="0204/5"/>
-<part name="R4" library="resistor" deviceset="R-EU_" device="0204/5"/>
-<part name="R5" library="resistor" deviceset="R-EU_" device="0204/5"/>
+<part name="R1" library="resistor" deviceset="R-EU_" device="0204/5" value="4,7 kOm"/>
+<part name="R2" library="resistor" deviceset="R-EU_" device="0204/5" value="4,7 kOm"/>
+<part name="R3" library="resistor" deviceset="R-EU_" device="0204/5" value="4,7 kOm"/>
+<part name="R4" library="resistor" deviceset="R-EU_" device="0204/5" value="4,7 kOm"/>
+<part name="R5" library="resistor" deviceset="R-EU_" device="0204/5" value="4,7 kOm"/>
 <part name="GND2" library="supply1" deviceset="GND" device=""/>
 <part name="P+3" library="supply1" deviceset="+5V" device=""/>
@@
 <part name="PAD31" library="wirepad" deviceset="WIREPAD" device="SMD1,27-254"/>
 <part name="PAD32" library="wirepad" deviceset="WIREPAD" device="SMD1,27-254"/>
-<part name="R6" library="resistor" deviceset="R-EU_" device="0204/2V"/>
-<part name="R7" library="resistor" deviceset="R-EU_" device="0204/2V"/>
-<part name="R8" library="resistor" deviceset="R-EU_" device="0204/2V"/>
-<part name="R9" library="resistor" deviceset="R-EU_" device="0204/2V"/>
-<part name="R10" library="resistor" deviceset="R-EU_" device="0204/2V"/>
+<part name="R6" library="resistor" deviceset="R-EU_" device="0204/2V" value="1 kOm"/>
+<part name="R7" library="resistor" deviceset="R-EU_" device="0204/2V" value="1 kOm"/>
+<part name="R8" library="resistor" deviceset="R-EU_" device="0204/2V" value="1 kOm"/>
+<part name="R9" library="resistor" deviceset="R-EU_" device="0204/2V" value="1 kOm"/>
+<part name="R10" library="resistor" deviceset="R-EU_" device="0204/2V" value="1 kOm"/>
 <part name="C1" library="resistor" deviceset="CPOL-EU" device="E2.5-5"/>
 <part name="C2" library="resistor" deviceset="CPOL-EU" device="E2.5-5"/>
