File: design_board/op_amp/op_amp.brd (EAGLE design)
At the start: 23.8 x 127.5 mm, 12 parts, among them IC1 LM393D

Commit message: Изменены платы controller.brd и relay.brd - скорректированы зазоры между платами, оp_amp.brd - добавлено отверстие для прокладки проводки между уровнями. Изменена схема сontroller.sch - добавлены номиналы резисторов обвязки оптопар.
Other:
- outline, holes or cut-outs redrawn
Changed lines of the file:
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@@
 <wire x1="45.75" y1="134" x2="22" y2="134" width="0.254" layer="20"/>
 <wire x1="22" y1="134" x2="22" y2="93" width="0.254" layer="20"/>
+<wire x1="24.75" y1="101" x2="43.25" y2="101" width="0.254" layer="20"/>
+<wire x1="43.25" y1="101" x2="43.25" y2="98.75" width="0.254" layer="20"/>
+<dimension x1="43.25" y1="101" x2="43.25" y2="98.75" x3="20.25" y3="99.875" textsize="1.778" layer="19"/>
+<wire x1="24.75" y1="101" x2="24.75" y2="98.75" width="0.254" layer="20"/>
+<wire x1="24.75" y1="98.75" x2="43.25" y2="98.75" width="0.254" layer="20"/>
 </plain>
 <attributes>
